Commit message: update urdf

File: urdf/pan_tilt_urdf.xacro (robot description, xacro)
@@ -6,14 +6,8 @@
 <xacro:include filename="$(find pan_tilt_ros)/urdf/pan_tilt_urdf.gazebo" />
 <link name="base_link">
-  <inertial>
-    <origin xyz="0.0 0.0 0.0" rpy="0 0 0"/>
-    <!--origin xyz="-0.0015531314926290208 -0.006917643689614827 0.01296710005093539" rpy="0 0 0"/ -->
-    <mass value="0.08629878221299303"/> <!-- y = 6.8392, x = 1.55..-->
-    <inertia ixx="9e-06" iyy="1e-05" izz="9e-06" ixy="-0.0" iyz="0.0" ixz="0.0"/>
-  </inertial>
   <visual>
     <origin xyz="0 0 0" rpy="0 0 0"/>
     <geometry>
-      <mesh filename="package://pan_tilt_ros/meshes/base_link.stl" scale="0.001 0.001 0.001"/>
+      <mesh filename="package://pan_tilt_ros/meshes/base_link.stl" scale="${stl_scale} ${stl_scale} ${stl_scale}"/>
     </geometry>
     <material name="silver"/>
@@ -22,11 +16,18 @@
     <origin xyz="0 0 0" rpy="0 0 0"/>
     <geometry>
-      <mesh filename="package://pan_tilt_ros/meshes/base_link.stl" scale="0.001 0.001 0.001"/>
+      <mesh filename="package://pan_tilt_ros/meshes/base_link.stl" scale="${stl_scale} ${stl_scale} ${stl_scale}"/>
     </geometry>
   </collision>
 </link>
+<link name="base_link_inertial">
+  <inertial>
+    <origin xyz="-0.0015531314926290208 -0.006917643689614827 0.01296710005093539" rpy="0 0 0"/>
+    <mass value="0.08629878221299303"/> <!-- y = 6.8392, x = 1.55..-->
+    <inertia ixx="9e-06" iyy="1e-05" izz="9e-06" ixy="-0.0" iyz="0.0" ixz="0.0"/>
+  </inertial>
+</link>
 <link name="tilt_motor">
   <inertial>
-    <origin xyz="0.016329668153777396 -0.004542288424019495 0.01025020002429897" rpy="0 0 0"/>
+    <!-- origin xyz="0.016329668153777396 -0.004542288424019495 0.01025020002429897" rpy="0 0 0"/ -->
     <mass value="0.05372359693747839"/>
     <inertia ixx="1.2e-05" iyy="7e-06" izz="1.3e-05" ixy="0.0" iyz="0.0" ixz="0.0"/>
@@ -35,5 +36,5 @@
     <origin xyz="0.017719 -0.005007 -0.0272" rpy="0 0 0"/>
     <geometry>
-      <mesh filename="package://pan_tilt_ros/meshes/st3215.stl" scale="0.001 0.001 0.001"/>
+      <mesh filename="package://pan_tilt_ros/meshes/st3215.stl" scale="${stl_scale} ${stl_scale} ${stl_scale}"/>
     </geometry>
     <material name="silver"/>
@@ -42,5 +43,5 @@
     <origin xyz="0.017719 -0.005007 -0.0272" rpy="0 0 0"/>
     <geometry>
-      <mesh filename="package://pan_tilt_ros/meshes/st3215.stl" scale="0.001 0.001 0.001"/>
+      <mesh filename="package://pan_tilt_ros/meshes/st3215.stl" scale="${stl_scale} ${stl_scale} ${stl_scale}"/>
     </geometry>
   </collision>
@@ -48,5 +49,5 @@
 <link name="pan_tilt_link">
   <inertial>
-    <origin xyz="-0.013649125671909021 -7.296148707217065e-07 0.019463753088211883" rpy="0 0 0"/>
+    <!-- origin xyz="-0.013649125671909021 -7.296148707217065e-07 0.019463753088211883" rpy="0 0 0"/ -->
     <mass value="0.05018544007475792"/>
     <inertia ixx="1.3e-05" iyy="2.4e-05" izz="1.5e-05" ixy="0.0" iyz="0.0" ixz="0.0"/>
@@ -55,5 +56,5 @@
     <origin xyz="-0.012681 -0.013307 -0.037451" rpy="0 0 0"/>
     <geometry>
-      <mesh filename="package://pan_tilt_ros/meshes/pan_tilt_link.stl" scale="0.001 0.001 0.001"/>
+      <mesh filename="package://pan_tilt_ros/meshes/pan_tilt_link.stl" scale="${stl_scale} ${stl_scale} ${stl_scale}"/>
     </geometry>
     <material name="silver"/>
@@ -62,5 +63,5 @@
     <origin xyz="-0.012681 -0.013307 -0.037451" rpy="0 0 0"/>
     <geometry>
-      <mesh filename="package://pan_tilt_ros/meshes/pan_tilt_link.stl" scale="0.001 0.001 0.001"/>
+      <mesh filename="package://pan_tilt_ros/meshes/pan_tilt_link.stl" scale="${stl_scale} ${stl_scale} ${stl_scale}"/>
     </geometry>
   </collision>
@@ -68,5 +69,5 @@
 <link name="pan_motor">
   <inertial>
-    <origin xyz="4.332570443822941e-07 -0.012842310722113068 0.0173701073619867" rpy="0 0 0"/>
+    <!-- origin xyz="4.332570443822941e-07 -0.012842310722113068 0.0173701073619867" rpy="0 0 0"/ -->
     <mass value="0.05372359236261105"/>
     <inertia ixx="1.3e-05" iyy="7e-06" izz="1.2e-05" ixy="0.0" iyz="-0.0" ixz="-0.0"/>
@@ -75,5 +76,5 @@
     <origin xyz="0.001444 -0.013306 -0.073751" rpy="0 0 0"/>
     <geometry>
-      <mesh filename="package://pan_tilt_ros/meshes/st3215.stl" scale="0.001 0.001 0.001"/>
+      <mesh filename="package://pan_tilt_ros/meshes/st3215.stl" scale="${stl_scale} ${stl_scale} ${stl_scale}"/>
     </geometry>
     <material name="silver"/>
@@ -82,5 +83,5 @@
     <origin xyz="0.001444 -0.013306 -0.073751" rpy="0 0 0"/>
     <geometry>
-      <mesh filename="package://pan_tilt_ros/meshes/st3215.stl" scale="0.001 0.001 0.001"/>
+      <mesh filename="package://pan_tilt_ros/meshes/st3215.stl" scale="${stl_scale} ${stl_scale} ${stl_scale}"/>
     </geometry>
   </collision>
@@ -88,5 +89,5 @@
 <link name="camera_link">
   <inertial>
-    <origin xyz="0.00705968500450624 -0.04297866937829162 -0.013250710871012955" rpy="0 0 0"/>
+    <!-- origin xyz="0.00705968500450624 -0.04297866937829162 -0.013250710871012955" rpy="0 0 0"/ -->
     <mass value="0.4069750331377844"/>
     <inertia ixx="0.00017" iyy="0.000299" izz="0.000309" ixy="2.8e-05" iyz="1.2e-05" ixz="-3e-06"/>
@@ -95,5 +96,5 @@
     <origin xyz="0.011694 -0.005005 -0.10745" rpy="0 0 0"/>
     <geometry>
-      <mesh filename="package://pan_tilt_ros/meshes/camera_link.stl" scale="0.001 0.001 0.001"/>
+      <mesh filename="package://pan_tilt_ros/meshes/camera_link.stl" scale="${stl_scale} ${stl_scale} ${stl_scale}"/>
     </geometry>
     <material name="silver"/>
@@ -102,5 +103,5 @@
     <origin xyz="0.011694 -0.005005 -0.10745" rpy="0 0 0"/>
     <geometry>
-      <mesh filename="package://pan_tilt_ros/meshes/camera_link.stl" scale="0.001 0.001 0.001"/>
+      <mesh filename="package://pan_tilt_ros/meshes/camera_link.stl" scale="${stl_scale} ${stl_scale} ${stl_scale}"/>
     </geometry>
   </collision>
@@ -108,5 +109,5 @@
 <link name="oakd">
   <inertial>
-    <origin xyz="-5.307190548554767e-07 -5.488642980319702e-06 1.1787927783890595e-07" rpy="0 0 0"/>
+    <!-- origin xyz="-5.307190548554767e-07 -5.488642980319702e-06 1.1787927783890595e-07" rpy="0 0 0"/ -->
     <mass value="6.165375582666816e-06"/>
     <inertia ixx="0.0" iyy="0.0" izz="0.0" ixy="0.0" iyz="0.0" ixz="0.0"/>
@@ -115,5 +116,5 @@
     <origin xyz="0.00237 0.059998 -0.105099" rpy="0 0 0"/>
     <geometry>
-      <mesh filename="package://pan_tilt_ros/meshes/oakd.stl" scale="0.001 0.001 0.001"/>
+      <mesh filename="package://pan_tilt_ros/meshes/oakd.stl" scale="${stl_scale} ${stl_scale} ${stl_scale}"/>
     </geometry>
     <material name="silver"/>
@@ -122,36 +123,41 @@
     <origin xyz="0.00237 0.059998 -0.105099" rpy="0 0 0"/>
     <geometry>
-      <mesh filename="package://pan_tilt_ros/meshes/oakd.stl" scale="0.001 0.001 0.001"/>
+      <mesh filename="package://pan_tilt_ros/meshes/oakd.stl" scale="${stl_scale} ${stl_scale} ${stl_scale}"/>
     </geometry>
   </collision>
 </link>
+<joint name="base_inertial_fixed" type="fixed">
+  <parent link="base_link"/>
+  <child link="base_link_inertial"/>
+  <origin xyz="0 0 0" rpy="0 0 0"/>
+</joint>
 <joint name="tilt_to_base" type="fixed">
-  <origin xyz="-0.017719 0.005007 0.0272" rpy="0 0 0"/>
   <parent link="base_link"/>
   <child link="tilt_motor"/>
+  <origin xyz="-0.017719 0.005007 0.0272" rpy="0 0 0"/>
 </joint>
 <joint name="tilt_joint" type="revolute">
-  <origin xyz="0.0304 0.0083 0.010251" rpy="0 0 0"/>
   <parent link="tilt_motor"/>
   <child link="pan_tilt_link"/>
+  <origin xyz="0.0304 0.0083 0.010251" rpy="0 0 0"/>
   <axis xyz="1.0 0.0 0.0"/>
   <limit lower="${-pi_by_two}" upper="${pi_by_two}" effort="${st3215_effort}" velocity="${st3215_maxvel}"/>
 </joint>
 <joint name="pan_joint" type="revolute">
-  <origin xyz="-0.014125 -1e-06 0.0363" rpy="0 0 0"/>
   <parent link="pan_tilt_link"/>
   <child link="pan_motor"/>
   <axis xyz="0.0 0.0 1.0"/>
+  <origin xyz="-0.014125 -1e-06 0.0363" rpy="0 0 0"/>
   <limit lower="${-pi_by_two}" upper="${pi_by_two}" effort="${st3215_effort}" velocity="${st3215_maxvel}"/>
 </joint>
 <joint name="camera_mount_to_motor" type="fixed">
-  <origin xyz="-0.01025 -0.008301 0.033699" rpy="0 0 0"/>
   <parent link="pan_motor"/>
   <child link="camera_link"/>
+  <origin xyz="-0.01025 -0.008301 0.033699" rpy="0 0 0"/>
 </joint>
 <joint name="camera_to_mount" type="fixed">
-  <origin xyz="0.009324 -0.065003 -0.002351" rpy="0 0 0"/>
   <parent link="camera_link"/>
   <child link="oakd"/>
+  <origin xyz="0.009324 -0.065003 -0.002351" rpy="0 0 0"/>
 </joint>
 </robot>

Commit message: Update pan_tilt_urdf.xacro

File: urdf/pan_tilt_urdf.xacro (robot description, xacro)
@@ -2,5 +2,4 @@
 <robot name="pan_tilt" xmlns:xacro="http://www.ros.org/wiki/xacro">
 <xacro:include filename="$(find pan_tilt_ros)/urdf/materials.xacro" />
-<xacro:include filename="$(find pan_tilt_ros)/urdf/pan_tilt_urdf.common" />
 <xacro:include filename="$(find pan_tilt_ros)/urdf/pan_tilt_urdf.trans" />
 <xacro:include filename="$(find pan_tilt_ros)/urdf/pan_tilt_urdf.gazebo" />
@@ -9,12 +8,12 @@
     <origin xyz="0 0 0" rpy="0 0 0"/>
     <geometry>
-      <mesh filename="package://pan_tilt_ros/meshes/base_link.stl" scale="${stl_scale} ${stl_scale} ${stl_scale}"/>
+      <mesh filename="package://pan_tilt_ros/meshes/base_link.stl" scale="0.001 0.001 0.001"/>
     </geometry>
-    <material name="silver"/>
+    <material name="matte_black"/>
   </visual>
   <collision>
     <origin xyz="0 0 0" rpy="0 0 0"/>
     <geometry>
-      <mesh filename="package://pan_tilt_ros/meshes/base_link.stl" scale="${stl_scale} ${stl_scale} ${stl_scale}"/>
+      <mesh filename="package://pan_tilt_ros/meshes/base_link.stl" scale="0.001 0.001 0.001"/>
     </geometry>
   </collision>
@@ -22,46 +21,46 @@
 <link name="base_link_inertial">
   <inertial>
-    <origin xyz="-0.0015531314926290208 -0.006917643689614827 0.01296710005093539" rpy="0 0 0"/>
-    <mass value="0.08629878221299303"/> <!-- y = 6.8392, x = 1.55..-->
-    <inertia ixx="9e-06" iyy="1e-05" izz="9e-06" ixy="-0.0" iyz="0.0" ixz="0.0"/>
+    <origin xyz="3.100257446207066e-05 -2.4988496235187414e-05 0.012657202544439227" rpy="0 0 0"/>
+    <mass value="0.08489188819476734"/>
+    <inertia ixx="1e-05" iyy="8e-06" izz="9e-06" ixy="-0.0" iyz="-0.0" ixz="-0.0"/>
   </inertial>
 </link>
 <link name="tilt_motor">
   <inertial>
-    <!-- origin xyz="0.016329668153777396 -0.004542288424019495 0.01025020002429897" rpy="0 0 0"/ -->
-    <mass value="0.05372359693747839"/>
-    <inertia ixx="1.2e-05" iyy="7e-06" izz="1.3e-05" ixy="0.0" iyz="0.0" ixz="0.0"/>
+    <origin xyz="-0.019875146307512716 0.0162793854605978 0.010245897629134384" rpy="0 0 0"/>
+    <mass value="0.04700597163076828"/>
+    <inertia ixx="6e-06" iyy="1e-05" izz="1.1e-05" ixy="-0.0" iyz="-0.0" ixz="0.0"/>
   </inertial>
   <visual>
-    <origin xyz="0.017719 -0.005007 -0.0272" rpy="0 0 0"/>
+    <origin xyz="-0.01243 0.016155 -0.0275" rpy="0 0 0"/>
     <geometry>
-      <mesh filename="package://pan_tilt_ros/meshes/st3215.stl" scale="${stl_scale} ${stl_scale} ${stl_scale}"/>
+      <mesh filename="package://pan_tilt_ros/meshes/tilt_motor.stl" scale="0.001 0.001 0.001"/>
     </geometry>
-    <material name="silver"/>
+    <material name="matte_black"/>
   </visual>
   <collision>
-    <origin xyz="0.017719 -0.005007 -0.0272" rpy="0 0 0"/>
+    <origin xyz="-0.01243 0.016155 -0.0275" rpy="0 0 0"/>
     <geometry>
-      <mesh filename="package://pan_tilt_ros/meshes/st3215.stl" scale="${stl_scale} ${stl_scale} ${stl_scale}"/>
+      <mesh filename="package://pan_tilt_ros/meshes/tilt_motor.stl" scale="0.001 0.001 0.001"/>
     </geometry>
   </collision>
 </link>
-<link name="pan_tilt_link">
+<link name="pan_tilt_bracket">
   <inertial>
-    <!-- origin xyz="-0.013649125671909021 -7.296148707217065e-07 0.019463753088211883" rpy="0 0 0"/ -->
-    <mass value="0.05018544007475792"/>
-    <inertia ixx="1.3e-05" iyy="2.4e-05" izz="1.5e-05" ixy="0.0" iyz="0.0" ixz="0.0"/>
+    <origin xyz="1.033653797971601e-09 -0.016649542795301807 0.019464379532745206" rpy="0 0 0"/>
+    <mass value="0.05018543913699325"/>
+    <inertia ixx="2.4e-05" iyy="1.3e-05" izz="1.5e-05" ixy="-0.0" iyz="0.0" ixz="0.0"/>
   </inertial>
   <visual>
-    <origin xyz="-0.012681 -0.013307 -0.037451" rpy="0 0 0"/>
+    <origin xyz="0.02032 -0.017545 -0.03775" rpy="0 0 0"/>
     <geometry>
-      <mesh filename="package://pan_tilt_ros/meshes/pan_tilt_link.stl" scale="${stl_scale} ${stl_scale} ${stl_scale}"/>
+      <mesh filename="package://pan_tilt_ros/meshes/pan_tilt_bracket.stl" scale="0.001 0.001 0.001"/>
     </geometry>
-    <material name="silver"/>
+    <material name="matte_black"/>
   </visual>
   <collision>
-    <origin xyz="-0.012681 -0.013307 -0.037451" rpy="0 0 0"/>
+    <origin xyz="0.02032 -0.017545 -0.03775" rpy="0 0 0"/>
     <geometry>
-      <mesh filename="package://pan_tilt_ros/meshes/pan_tilt_link.stl" scale="${stl_scale} ${stl_scale} ${stl_scale}"/>
+      <mesh filename="package://pan_tilt_ros/meshes/pan_tilt_bracket.stl" scale="0.001 0.001 0.001"/>
     </geometry>
   </collision>
@@ -69,19 +68,19 @@
 <link name="pan_motor">
   <inertial>
-    <!-- origin xyz="4.332570443822941e-07 -0.012842310722113068 0.0173701073619867" rpy="0 0 0"/ -->
-    <mass value="0.05372359236261105"/>
-    <inertia ixx="1.3e-05" iyy="7e-06" izz="1.2e-05" ixy="0.0" iyz="-0.0" ixz="-0.0"/>
+    <origin xyz="0.012874853692487125 -4.173783098805313e-06 0.0174208176028941" rpy="0 0 0"/>
+    <mass value="0.04700597163076828"/>
+    <inertia ixx="6e-06" iyy="1.1e-05" izz="1e-05" ixy="0.0" iyz="0.0" ixz="0.0"/>
   </inertial>
   <visual>
-    <origin xyz="0.001444 -0.013306 -0.073751" rpy="0 0 0"/>
+    <origin xyz="0.02032 -0.00042 -0.07405" rpy="0 0 0"/>
     <geometry>
-      <mesh filename="package://pan_tilt_ros/meshes/st3215.stl" scale="${stl_scale} ${stl_scale} ${stl_scale}"/>
+      <mesh filename="package://pan_tilt_ros/meshes/pan_motor.stl" scale="0.001 0.001 0.001"/>
     </geometry>
-    <material name="silver"/>
+    <material name="matte_black"/>
   </visual>
   <collision>
-    <origin xyz="0.001444 -0.013306 -0.073751" rpy="0 0 0"/>
+    <origin xyz="0.02032 -0.00042 -0.07405" rpy="0 0 0"/>
     <geometry>
-      <mesh filename="package://pan_tilt_ros/meshes/st3215.stl" scale="${stl_scale} ${stl_scale} ${stl_scale}"/>
+      <mesh filename="package://pan_tilt_ros/meshes/pan_motor.stl" scale="0.001 0.001 0.001"/>
     </geometry>
   </collision>
@@ -89,19 +88,19 @@
 <link name="camera_link">
   <inertial>
-    <!-- origin xyz="0.00705968500450624 -0.04297866937829162 -0.013250710871012955" rpy="0 0 0"/ -->
-    <mass value="0.4069750331377844"/>
-    <inertia ixx="0.00017" iyy="0.000299" izz="0.000309" ixy="2.8e-05" iyz="1.2e-05" ixz="-3e-06"/>
+    <origin xyz="-0.004991360468491857 -0.011542339627033346 0.004227044433613547" rpy="0 0 0"/>
+    <mass value="0.09449139072993021"/>
+    <inertia ixx="2.1e-05" iyy="1.8e-05" izz="2.1e-05" ixy="-6e-06" iyz="0.0" ixz="0.0"/>
   </inertial>
   <visual>
-    <origin xyz="0.011694 -0.005005 -0.10745" rpy="0 0 0"/>
+    <origin xyz="-0.014736 -0.00042 -0.08975" rpy="0 0 0"/>
     <geometry>
-      <mesh filename="package://pan_tilt_ros/meshes/camera_link.stl" scale="${stl_scale} ${stl_scale} ${stl_scale}"/>
+      <mesh filename="package://pan_tilt_ros/meshes/camera_link.stl" scale="0.001 0.001 0.001"/>
     </geometry>
-    <material name="silver"/>
+    <material name="matte_black"/>
   </visual>
   <collision>
-    <origin xyz="0.011694 -0.005005 -0.10745" rpy="0 0 0"/>
+    <origin xyz="-0.014736 -0.00042 -0.08975" rpy="0 0 0"/>
     <geometry>
-      <mesh filename="package://pan_tilt_ros/meshes/camera_link.stl" scale="${stl_scale} ${stl_scale} ${stl_scale}"/>
+      <mesh filename="package://pan_tilt_ros/meshes/camera_link.stl" scale="0.001 0.001 0.001"/>
     </geometry>
   </collision>
@@ -109,55 +108,53 @@
 <link name="oakd">
   <inertial>
-    <!-- origin xyz="-5.307190548554767e-07 -5.488642980319702e-06 1.1787927783890595e-07" rpy="0 0 0"/ -->
-    <mass value="6.165375582666816e-06"/>
-    <inertia ixx="0.0" iyy="0.0" izz="0.0" ixy="0.0" iyz="0.0" ixz="0.0"/>
+    <origin xyz="0.01740685213679074 0.0005740020595517798 0.007939642786094867" rpy="0 0 0"/>
+    <mass value="0.3193880841082503"/>
+    <inertia ixx="0.000275" iyy="9.8e-05" izz="0.000232" ixy="-1e-06" iyz="-0.0" ixz="-5e-06"/>
   </inertial>
   <visual>
-    <origin xyz="0.00237 0.059998 -0.105099" rpy="0 0 0"/>
+    <origin xyz="-0.019836 8e-05 -0.08971" rpy="0 0 0"/>
     <geometry>
-      <mesh filename="package://pan_tilt_ros/meshes/oakd.stl" scale="${stl_scale} ${stl_scale} ${stl_scale}"/>
+      <mesh filename="package://pan_tilt_ros/meshes/oakd.stl" scale="0.001 0.001 0.001"/>
     </geometry>
-    <material name="silver"/>
+    <material name="matte_black"/>
   </visual>
   <collision>
-    <origin xyz="0.00237 0.059998 -0.105099" rpy="0 0 0"/>
+    <origin xyz="-0.019836 8e-05 -0.08971" rpy="0 0 0"/>
     <geometry>
-      <mesh filename="package://pan_tilt_ros/meshes/oakd.stl" scale="${stl_scale} ${stl_scale} ${stl_scale}"/>
+      <mesh filename="package://pan_tilt_ros/meshes/oakd.stl" scale="0.001 0.001 0.001"/>
     </geometry>
   </collision>
 </link>
 <joint name="base_inertial_fixed" type="fixed">
+  <origin xyz="0 0 0" rpy="0 0 0"/>
   <parent link="base_link"/>
   <child link="base_link_inertial"/>
-  <origin xyz="0 0 0" rpy="0 0 0"/>
 </joint>
-<joint name="tilt_to_base" type="fixed">
+<joint name="base_tilt_fixed" type="fixed">
+  <origin xyz="0.01243 -0.016155 0.0275" rpy="0 0 0"/>
   <parent link="base_link"/>
   <child link="tilt_motor"/>
-  <origin xyz="-0.017719 0.005007 0.0272" rpy="0 0 0"/>
 </joint>
-<joint name="tilt_joint" type="revolute">
+<joint name="tilt_joint" type="continuous">
+  <origin xyz="-0.03275 0.0337 0.01025" rpy="0 0 0"/>
   <parent link="tilt_motor"/>
-  <child link="pan_tilt_link"/>
-  <origin xyz="0.0304 0.0083 0.010251" rpy="0 0 0"/>
-  <axis xyz="1.0 0.0 0.0"/>
-  <limit lower="${-pi_by_two}" upper="${pi_by_two}" effort="${st3215_effort}" velocity="${st3215_maxvel}"/>
+  <child link="pan_tilt_bracket"/>
+  <axis xyz="-0.0 1.0 0.0"/>
 </joint>
-<joint name="pan_joint" type="revolute">
-  <parent link="pan_tilt_link"/>
+<joint name="pan_joint" type="continuous">
+  <origin xyz="0.0 -0.017125 0.0363" rpy="0 0 0"/>
+  <parent link="pan_tilt_bracket"/>
   <child link="pan_motor"/>
   <axis xyz="0.0 0.0 1.0"/>
-  <origin xyz="-0.014125 -1e-06 0.0363" rpy="0 0 0"/>
-  <limit lower="${-pi_by_two}" upper="${pi_by_two}" effort="${st3215_effort}" velocity="${st3215_maxvel}"/>
 </joint>
-<joint name="camera_mount_to_motor" type="fixed">
+<joint name="pan_mount_fixed" type="fixed">
+  <origin xyz="0.035056 0.0 0.0157" rpy="0 0 0"/>
   <parent link="pan_motor"/>
   <child link="camera_link"/>
-  <origin xyz="-0.01025 -0.008301 0.033699" rpy="0 0 0"/>
 </joint>
-<joint name="camera_to_mount" type="fixed">
+<joint name="mount_camera_fixed" type="fixed">
+  <origin xyz="0.0051 -0.0005 -4e-05" rpy="0 0 0"/>
   <parent link="camera_link"/>
   <child link="oakd"/>
-  <origin xyz="0.009324 -0.065003 -0.002351" rpy="0 0 0"/>
 </joint>
 </robot>

Commit message: Update pan_tilt_urdf.xacro

File: urdf/pan_tilt_urdf.xacro (robot description, xacro)
@@ -86,5 +86,5 @@
   </collision>
 </link>
-<link name="camera_link">
+<link name="payload_link">
   <inertial>
     <origin xyz="-0.004991360468491857 -0.011542339627033346 0.004227044433613547" rpy="0 0 0"/>
@@ -95,5 +95,5 @@
     <origin xyz="-0.014736 -0.00042 -0.08975" rpy="0 0 0"/>
     <geometry>
-      <mesh filename="package://pan_tilt_ros/meshes/camera_link.stl" scale="0.001 0.001 0.001"/>
+      <mesh filename="package://pan_tilt_ros/meshes/payload_link.stl" scale="0.001 0.001 0.001"/>
     </geometry>
     <material name="matte_black"/>
@@ -102,25 +102,5 @@
     <origin xyz="-0.014736 -0.00042 -0.08975" rpy="0 0 0"/>
     <geometry>
-      <mesh filename="package://pan_tilt_ros/meshes/camera_link.stl" scale="0.001 0.001 0.001"/>
-    </geometry>
-  </collision>
-</link>
-<link name="oakd">
-  <inertial>
-    <origin xyz="0.01740685213679074 0.0005740020595517798 0.007939642786094867" rpy="0 0 0"/>
-    <mass value="0.3193880841082503"/>
-    <inertia ixx="0.000275" iyy="9.8e-05" izz="0.000232" ixy="-1e-06" iyz="-0.0" ixz="-5e-06"/>
-  </inertial>
-  <visual>
-    <origin xyz="-0.019836 8e-05 -0.08971" rpy="0 0 0"/>
-    <geometry>
-      <mesh filename="package://pan_tilt_ros/meshes/oakd.stl" scale="0.001 0.001 0.001"/>
-    </geometry>
-    <material name="matte_black"/>
-  </visual>
-  <collision>
-    <origin xyz="-0.019836 8e-05 -0.08971" rpy="0 0 0"/>
-    <geometry>
-      <mesh filename="package://pan_tilt_ros/meshes/oakd.stl" scale="0.001 0.001 0.001"/>
+      <mesh filename="package://pan_tilt_ros/meshes/payload_link.stl" scale="0.001 0.001 0.001"/>
     </geometry>
   </collision>
@@ -148,13 +128,8 @@
   <axis xyz="0.0 0.0 1.0"/>
 </joint>
-<joint name="pan_mount_fixed" type="fixed">
+<joint name="payload_mount_fixed" type="fixed">
   <origin xyz="0.035056 0.0 0.0157" rpy="0 0 0"/>
   <parent link="pan_motor"/>
-  <child link="camera_link"/>
-</joint>
-<joint name="mount_camera_fixed" type="fixed">
-  <origin xyz="0.0051 -0.0005 -4e-05" rpy="0 0 0"/>
-  <parent link="camera_link"/>
-  <child link="oakd"/>
+  <child link="payload_link"/>
 </joint>
 </robot>

Commit message: update config and URDF

File: urdf/pan_tilt_urdf.xacro (robot description, xacro)
@@ -93,5 +93,5 @@
   </inertial>
   <visual>
-    <origin xyz="-0.014736 -0.00042 -0.08975" rpy="0 0 0"/>
+    <origin xyz="-0.0001099 0.0164388 -0.0939786" rpy="0 0 0"/>
     <geometry>
       <mesh filename="package://pan_tilt_ros/meshes/payload_link.stl" scale="0.001 0.001 0.001"/>
@@ -100,5 +100,5 @@
   </visual>
   <collision>
-    <origin xyz="-0.014736 -0.00042 -0.08975" rpy="0 0 0"/>
+    <origin xyz="-0.0001099 0.0164388 -0.0939786" rpy="0 0 0"/>
     <geometry>
       <mesh filename="package://pan_tilt_ros/meshes/payload_link.stl" scale="0.001 0.001 0.001"/>
@@ -129,5 +129,5 @@
 </joint>
 <joint name="payload_mount_fixed" type="fixed">
-  <origin xyz="0.035056 0.0 0.0157" rpy="0 0 0"/>
+  <origin xyz="0.0204299 -0.0168588 0.0199286" rpy="0 0 0"/>
   <parent link="pan_motor"/>
   <child link="payload_link"/>
